File: Seck_C_75.kicad_pcb (KiCad board)
At the start: 2 copper layers, 285 x 94.6 mm, 122 parts, among them SW1 RESET, U1 ATmega32U4-AU, Y1 16MHz

Commit message: Layout
Parts:
- removed K_0: KC_ESC, MX_Only:MXOnly-1U-NoLED
- removed K_013A1: KC_BSPC, MX_Only:MXOnly-1U-NoLED
- removed K_100: KC_TAB, MX_Only:MXOnly-1.5U-NoLED
- removed K_101: KC_Q, MX_Only:MXOnly-1U-NoLED
- removed K_102: KC_W, MX_Only:MXOnly-1U-NoLED
- removed K_103: KC_E, MX_Only:MXOnly-1U-NoLED
- removed K_104: KC_R, MX_Only:MXOnly-1U-NoLED
- removed K_105: KC_T, MX_Only:MXOnly-1U-NoLED
- removed K_106: KC_Y, MX_Only:MXOnly-1U-NoLED
- removed K_107: KC_U, MX_Only:MXOnly-1U-NoLED
- removed K_108: KC_I, MX_Only:MXOnly-1U-NoLED
- removed K_109: KC_O, MX_Only:MXOnly-1U-NoLED
- removed K_110: KC_P, MX_Only:MXOnly-1U-NoLED
- removed K_111: KC_LBRC, MX_Only:MXOnly-1U-NoLED
- removed K_112: KC_RBRC, MX_Only:MXOnly-1U-NoLED
- removed K_113: KC_BSLS, MX_Only:MXOnly-1.5U-NoLED
- removed K_200: KC_CAPS, MX_Only:MXOnly-1.75U-NoLED
- removed K_200A1: KC_CAPS, MX_Only:MXOnly-1.25U-NoLED
- removed K_201: KC_A, MX_Only:MXOnly-1U-NoLED
- removed K_202: KC_S, MX_Only:MXOnly-1U-NoLED
- removed K_203: KC_D, MX_Only:MXOnly-1U-NoLED
- removed K_204: KC_F, MX_Only:MXOnly-1U-NoLED
- removed K_205: KC_G, MX_Only:MXOnly-1U-NoLED
- removed K_206: KC_H, MX_Only:MXOnly-1U-NoLED
- removed K_207: KC_J, MX_Only:MXOnly-1U-NoLED
- removed K_208: KC_K, MX_Only:MXOnly-1U-NoLED
- removed K_209: KC_L, MX_Only:MXOnly-1U-NoLED
- removed K_210: KC_SCLN, MX_Only:MXOnly-1U-NoLED
- removed K_211: KC_QUOT, MX_Only:MXOnly-1U-NoLED
- removed K_212: KC_ENT, MX_Only:MXOnly-2.25U-NoLED
- removed K_213: KC_DEL, MX_Only:MXOnly-1U-NoLED
- removed K_300: KC_LSFT, MX_Only:MXOnly-2.25U-NoLED
- removed K_301: KC_Z, MX_Only:MXOnly-1U-NoLED
- removed K_302: KC_X, MX_Only:MXOnly-1U-NoLED
- removed K_303: KC_C, MX_Only:MXOnly-1U-NoLED
- removed K_304: KC_V, MX_Only:MXOnly-1U-NoLED
- removed K_305: KC_B, MX_Only:MXOnly-1U-NoLED
- removed K_306: KC_N, MX_Only:MXOnly-1U-NoLED
- removed K_307: KC_M, MX_Only:MXOnly-1U-NoLED
- removed K_308: KC_COMM, MX_Only:MXOnly-1U-NoLED
- removed K_309: KC_DOT, MX_Only:MXOnly-1U-NoLED
- removed K_310: KC_SLSH, MX_Only:MXOnly-1U-NoLED
- removed K_311: KC_RSFT, MX_Only:MXOnly-2.75U-NoLED
- removed K_311A1: KC_RSFT, MX_Only:MXOnly-1.75U-NoLED
- removed K_312, K_410A1: KC_MO(1), MX_Only:MXOnly-1U-NoLED
- removed K_400: KC_LCTL, MX_Only:MXOnly-1.25U-NoLED
- removed K_400A1: KC_LCTL, MX_Only:MXOnly-1.5U-NoLED
- removed K_401: KC_LGUI, MX_Only:MXOnly-1.25U-NoLED
- removed K_401A1: KC_LGUI, MX_Only:MXOnly-1U-NoLED
- removed K_402: KC_LALT, MX_Only:MXOnly-1.25U-NoLED
- removed K_402A1: KC_LALT, MX_Only:MXOnly-1.5U-NoLED
- removed K_406: KC_SPC, MX_Only:MXOnly-6.25U-ReversedStabilizers-NoLED
- removed K_406A1: KC_SPC, MX_Only:MXOnly-7U-ReversedStabilizers-NoLED
- removed K_408: KC_RALT, MX_Only:MXOnly-1.25U-NoLED
- removed K_409: KC_RGUI, MX_Only:MXOnly-1.25U-NoLED
- removed K_409A1: KC_RALT, MX_Only:MXOnly-1.5U-NoLED
- removed K_410: KC_MO(1), MX_Only:MXOnly-1.25U-NoLED
- removed K_411: KC_RCTL, MX_Only:MXOnly-1.25U-NoLED
- removed K_411A1: KC_RCTL, MX_Only:MXOnly-1.5U-NoLED
- added D33: D_Small, Custom_Footprints:D_SOD-123_Annotated, F.Cu at (-58.3, 21.7)
- added D34: D_Small, Custom_Footprints:D_SOD-123_Annotated, F.Cu at (-61.7, 93.3)
- added D35: D_Small, Custom_Footprints:D_SOD-123_Annotated, F.Cu at (-65.1, 87.5)
- added D36: D_Small, Custom_Footprints:D_SOD-123_Annotated, F.Cu at (-68.4, 87.5)
- added D37: D_Small, Custom_Footprints:D_SOD-123_Annotated, F.Cu at (-65.1, 93.3)
- added D38: D_Small, Custom_Footprints:D_SOD-123_Annotated, F.Cu at (-58.4, 99.0)
- added D39: D_Small, Custom_Footprints:D_SOD-123_Annotated, F.Cu at (-65.0, 21.7)
- added D40: D_Small, Custom_Footprints:D_SOD-123_Annotated, F.Cu at (-68.3, 21.7)
- added D41: D_Small, Custom_Footprints:D_SOD-123_Annotated, F.Cu at (-71.7, 21.7)
- added D42: D_Small, Custom_Footprints:D_SOD-123_Annotated, F.Cu at (-71.8, 81.8)
- added D43: D_Small, Custom_Footprints:D_SOD-123_Annotated, F.Cu at (-61.7, 70.3)
- added D44: D_Small, Custom_Footprints:D_SOD-123_Annotated, F.Cu at (-62.2, 38.3)
- added D45: D_Small, Custom_Footprints:D_SOD-123_Annotated, F.Cu at (-64.5, 11.7)
- added D46: D_Small, Custom_Footprints:D_SOD-123_Annotated, F.Cu at (-67.9, 11.7)
- added D47: D_Small, Custom_Footprints:D_SOD-123_Annotated, F.Cu at (-71.2, 11.7)
- added D48: D_Small, Custom_Footprints:D_SOD-123_Annotated, F.Cu at (-58.4, 104.8)
- added D49: D_Small, Custom_Footprints:D_SOD-123_Annotated, F.Cu at (-58.4, 110.5)
- added D50: D_Small, Custom_Footprints:D_SOD-123_Annotated, F.Cu at (-61.7, 99.0)
- added D51: D_Small, Custom_Footprints:D_SOD-123_Annotated, F.Cu at (-61.7, 104.8)
- added D52: D_Small, Custom_Footprints:D_SOD-123_Annotated, F.Cu at (-68.4, 110.5)
- added D53: D_Small, Custom_Footprints:D_SOD-123_Annotated, F.Cu at (-65.1, 99.0)
- added D54: D_Small, Custom_Footprints:D_SOD-123_Annotated, F.Cu at (-61.2, 11.7)
- added D55: D_Small, Custom_Footprints:D_SOD-123_Annotated, F.Cu at (-68.4, 93.3)
- added D56: D_Small, Custom_Footprints:D_SOD-123_Annotated, F.Cu at (-68.4, 99.0)
- added D57: D_Small, Custom_Footprints:D_SOD-123_Annotated, F.Cu at (-71.8, 87.5)
- added D58: D_Small, Custom_Footprints:D_SOD-123_Annotated, F.Cu at (-71.8, 93.3)
- added D59: D_Small, Custom_Footprints:D_SOD-123_Annotated, F.Cu at (-58.8, 38.3)
- added D60: D_Small, Custom_Footprints:D_SOD-123_Annotated, F.Cu at (-71.8, 99.0)
- added D61: D_Small, Custom_Footprints:D_SOD-123_Annotated, F.Cu at (-68.4, 104.8)
- added D62: D_Small, Custom_Footprints:D_SOD-123_Annotated, F.Cu at (-65.1, 110.5)
- added D63: D_Small, Custom_Footprints:D_SOD-123_Annotated, F.Cu at (-61.7, 110.5)
- added D64: D_Small, Custom_Footprints:D_SOD-123_Annotated, F.Cu at (-71.8, 127.8)
- added D65: D_Small, Custom_Footprints:D_SOD-123_Annotated, F.Cu at (-58.4, 116.3)
- added D66: D_Small, Custom_Footprints:D_SOD-123_Annotated, F.Cu at (-61.7, 116.3)
- added D67: D_Small, Custom_Footprints:D_SOD-123_Annotated, F.Cu at (-58.4, 122.0)
- added D68: D_Small, Custom_Footprints:D_SOD-123_Annotated, F.Cu at (-71.8, 110.5)
- added D69: D_Small, Custom_Footprints:D_SOD-123_Annotated, F.Cu at (-71.8, 122.0)
- added D70: D_Small, Custom_Footprints:D_SOD-123_Annotated, F.Cu at (-58.4, 127.8)
- added D71: D_Small, Custom_Footprints:D_SOD-123_Annotated, F.Cu at (-61.7, 122.0)
- added D72: D_Small, Custom_Footprints:D_SOD-123_Annotated, F.Cu at (-65.1, 116.3)
- added D73: D_Small, Custom_Footprints:D_SOD-123_Annotated, F.Cu at (-62.1, 32.5)
- added D74: D_Small, Custom_Footprints:D_SOD-123_Annotated, F.Cu at (-68.4, 116.3)
- added D75: D_Small, Custom_Footprints:D_SOD-123_Annotated, F.Cu at (-71.8, 104.8)
- added D76: D_Small, Custom_Footprints:D_SOD-123_Annotated, F.Cu at (-68.4, 127.8)
- added D77: D_Small, Custom_Footprints:D_SOD-123_Annotated, F.Cu at (-74.6, 11.7)
- added D78: D_Small, Custom_Footprints:D_SOD-123_Annotated, F.Cu at (-68.4, 122.0)
- added D79: D_Small, Custom_Footprints:D_SOD-123_Annotated, F.Cu at (-65.1, 127.8)
- added D80: D_Small, Custom_Footprints:D_SOD-123_Annotated, F.Cu at (-71.8, 116.3)
- added D81: D_Small, Custom_Footprints:D_SOD-123_Annotated, F.Cu at (-61.7, 127.8)
- added D82: D_Small, Custom_Footprints:D_SOD-123_Annotated, F.Cu at (-65.1, 122.0)
- added J1: OLED, Custom_Footprints:SSD1306_OLED, F.Cu at (297.7, 19.8)
- added K_113A1: KC_BSPC, MX_Only:MXOnly-1U-NoLED, F.Cu at (269.1, 43.7)
- added K_14: KC_GRV, MX_Only:MXOnly-1U-NoLED, F.Cu at (21.4, 43.7)
- added K_15: KC_1, MX_Only:MXOnly-1U-NoLED, F.Cu at (40.5, 43.7)
- added K_16: KC_2, MX_Only:MXOnly-1U-NoLED, F.Cu at (59.5, 43.7)
- added K_17: KC_3, MX_Only:MXOnly-1U-NoLED, F.Cu at (78.6, 43.7)
- added K_18: KC_4, MX_Only:MXOnly-1U-NoLED, F.Cu at (97.6, 43.7)
- added K_19: KC_5, MX_Only:MXOnly-1U-NoLED, F.Cu at (116.7, 43.7)
- added K_20: KC_6, MX_Only:MXOnly-1U-NoLED, F.Cu at (135.7, 43.7)
- added K_21: KC_7, MX_Only:MXOnly-1U-NoLED, F.Cu at (154.8, 43.7)
- added K_22: KC_8, MX_Only:MXOnly-1U-NoLED, F.Cu at (173.8, 43.7)
- added K_23: KC_9, MX_Only:MXOnly-1U-NoLED, F.Cu at (192.9, 43.7)
- added K_24: KC_0, MX_Only:MXOnly-1U-NoLED, F.Cu at (211.9, 43.7)
- added K_25: KC_MINS, MX_Only:MXOnly-1U-NoLED, F.Cu at (231.0, 43.7)
- added K_26: KC_EQL, MX_Only:MXOnly-1U-NoLED, F.Cu at (250.0, 43.7)
- added K_27: KC_BSPC, MX_Only:MXOnly-2U-NoLED, F.Cu at (278.6, 43.7)
- added K_28: KC_DEL, MX_Only:MXOnly-1U-NoLED, F.Cu at (307.2, 43.7)
- added K_29: KC_TAB, MX_Only:MXOnly-1.5U-NoLED, F.Cu at (26.2, 62.7)
- added K_30: KC_Q, MX_Only:MXOnly-1U-NoLED, F.Cu at (50.0, 62.7)
- added K_300A1: KC_CAPS, MX_Only:MXOnly-1.25U-NoLED, F.Cu at (23.8, 81.8)
- added K_31: KC_W, MX_Only:MXOnly-1U-NoLED, F.Cu at (69.1, 62.7)
- added K_32: KC_E, MX_Only:MXOnly-1U-NoLED, F.Cu at (88.1, 62.7)
- added K_33: KC_R, MX_Only:MXOnly-1U-NoLED, F.Cu at (107.2, 62.7)
- added K_34: KC_T, MX_Only:MXOnly-1U-NoLED, F.Cu at (126.2, 62.7)
- added K_35: KC_Y, MX_Only:MXOnly-1U-NoLED, F.Cu at (145.3, 62.7)
- added K_36: KC_U, MX_Only:MXOnly-1U-NoLED, F.Cu at (164.3, 62.7)
- added K_37: KC_I, MX_Only:MXOnly-1U-NoLED, F.Cu at (183.4, 62.7)
- added K_38: KC_O, MX_Only:MXOnly-1U-NoLED, F.Cu at (202.4, 62.7)
- added K_39: KC_P, MX_Only:MXOnly-1U-NoLED, F.Cu at (221.5, 62.7)
- added K_40: KC_LBRC, MX_Only:MXOnly-1U-NoLED, F.Cu at (240.5, 62.7)
- added K_41: KC_RBRC, MX_Only:MXOnly-1U-NoLED, F.Cu at (259.6, 62.7)
- added K_42: KC_BSLS, MX_Only:MXOnly-1.5U-NoLED, F.Cu at (283.4, 62.7)
- added K_43: KC_INS, MX_Only:MXOnly-1U-NoLED, F.Cu at (307.2, 62.7)
- added K_44: KC_CAPS, MX_Only:MXOnly-1.75U-NoLED, F.Cu at (28.6, 81.8)
- added K_45: KC_A, MX_Only:MXOnly-1U-NoLED, F.Cu at (54.8, 81.8)
- added K_46: KC_S, MX_Only:MXOnly-1U-NoLED, F.Cu at (73.8, 81.8)
- added K_47: KC_D, MX_Only:MXOnly-1U-NoLED, F.Cu at (92.9, 81.8)
- added K_48: KC_F, MX_Only:MXOnly-1U-NoLED, F.Cu at (111.9, 81.8)
- added K_49: KC_G, MX_Only:MXOnly-1U-NoLED, F.Cu at (131.0, 81.8)
- added K_50: KC_H, MX_Only:MXOnly-1U-NoLED, F.Cu at (150.0, 81.8)
- added K_508A1: KC_, MX_Only:MXOnly-1.5U-NoLED, F.Cu at (216.7, 119.9)
- added K_51: KC_J, MX_Only:MXOnly-1U-NoLED, F.Cu at (169.1, 81.8)
- added K_510A1: KC_RCTL, MX_Only:MXOnly-1.5U-NoLED, F.Cu at (245.3, 119.9)
- added K_52: KC_K, MX_Only:MXOnly-1U-NoLED, F.Cu at (188.1, 81.8)
- added K_53: KC_L, MX_Only:MXOnly-1U-NoLED, F.Cu at (207.2, 81.8)
- added K_54: KC_SCLN, MX_Only:MXOnly-1U-NoLED, F.Cu at (226.2, 81.8)
- added K_55: KC_QUOT, MX_Only:MXOnly-1U-NoLED, F.Cu at (245.3, 81.8)
- added K_56: KC_ENT, MX_Only:MXOnly-2.25U-NoLED, F.Cu at (276.2, 81.8)
- added K_57: KC_BSLS, MX_Only:MXOnly-1U-NoLED, F.Cu at (288.1, 43.7)
- added K_58: KC_HOME, MX_Only:MXOnly-1U-NoLED, F.Cu at (307.2, 81.8)
- added K_59: KC_LSFT, MX_Only:MXOnly-2.25U-NoLED, F.Cu at (33.3, 100.8)
- added K_60: KC_Z, MX_Only:MXOnly-1U-NoLED, F.Cu at (64.3, 100.8)
- added K_61: KC_X, MX_Only:MXOnly-1U-NoLED, F.Cu at (83.3, 100.8)
- added K_62: KC_C, MX_Only:MXOnly-1U-NoLED, F.Cu at (102.4, 100.8)
- added K_63: KC_V, MX_Only:MXOnly-1U-NoLED, F.Cu at (121.4, 100.8)
- added K_64: KC_B, MX_Only:MXOnly-1U-NoLED, F.Cu at (140.5, 100.8)
- added K_65: KC_N, MX_Only:MXOnly-1U-NoLED, F.Cu at (159.5, 100.8)
- added K_66: KC_M, MX_Only:MXOnly-1U-NoLED, F.Cu at (178.6, 100.8)
- added K_67: KC_COMM, MX_Only:MXOnly-1U-NoLED, F.Cu at (197.6, 100.8)
- added K_68: KC_DOT, MX_Only:MXOnly-1U-NoLED, F.Cu at (216.7, 100.8)
- added K_69: KC_SLSH, MX_Only:MXOnly-1U-NoLED, F.Cu at (235.7, 100.8)
- added K_70: KC_RSFT, MX_Only:MXOnly-1.75U-NoLED, F.Cu at (261.9, 100.8)
- added K_71: KC_UP, MX_Only:MXOnly-1U-NoLED, F.Cu at (288.1, 100.8)
- added K_72: KC_END, MX_Only:MXOnly-1U-NoLED, F.Cu at (307.2, 100.8)
- added K_73: KC_LCTL, MX_Only:MXOnly-1.25U-NoLED, F.Cu at (23.8, 119.9)
- added K_74: KC_LGUI, MX_Only:MXOnly-1.25U-NoLED, F.Cu at (47.6, 119.9)
- added K_75: KC_LALT, MX_Only:MXOnly-1.25U-NoLED, F.Cu at (71.4, 119.9)
- added K_76: KC_SPC, MX_Only:MXOnly-6.25U-ReversedStabilizers-NoLED, F.Cu at (142.9, 119.9)
- added K_77: KC_RALT, MX_Only:MXOnly-1U-NoLED, F.Cu at (211.9, 119.9)
- added K_78: KC_RGUI, MX_Only:MXOnly-1U-NoLED, F.Cu at (231.0, 119.9)
- added K_79: KC_RCTL, MX_Only:MXOnly-1U-NoLED, F.Cu at (250.0, 119.9)
- added K_80: KC_LEFT, MX_Only:MXOnly-1U-NoLED, F.Cu at (269.1, 119.9)
- added K_81: KC_DOWN, MX_Only:MXOnly-1U-NoLED, F.Cu at (288.1, 119.9)
- added K_82: KC_RGHT, MX_Only:MXOnly-1U-NoLED, F.Cu at (307.2, 119.9)
- C1, C2, C3, C4, C5, ESD1, F1, R1, R2, R3, R4, R5, R6, SW1, U1, USB1, Y1: moved to F.Cu
- D1, D10, D11, D12, D13, D14, D15, D16, D17, D18, D19, D2, D20, D21, D22, D23, D24, D25, D26, D27, D28, D29, D3, D30, D31, D32, D4, D5, D6, D7, D8, D9: value BAV70 -> D_Small; footprint Custom_Footprints:SOT-23_Annotated -> Custom_Footprints:D_SOD-123_Annotated; moved to F.Cu
- K_1: value KC_1 -> KC_ESC
- K_10: value KC_0 -> KC_F9
- K_11: value KC_MINS -> KC_F10
- K_12: value KC_EQL -> KC_F11
- K_13: value KC_BSPC -> KC_F12; footprint MX_Only:MXOnly-2U-NoLED -> MX_Only:MXOnly-1U-NoLED
- K_2: value KC_2 -> KC_F1
- K_3: value KC_3 -> KC_F2
- K_4: value KC_4 -> KC_F3
- K_5: value KC_5 -> KC_F4
- K_6: value KC_6 -> KC_F5
- K_7: value KC_7 -> KC_F6
- K_8: value KC_8 -> KC_F7
- K_9: value KC_9 -> KC_F8
- moved D21 333.9 mm to (-71.8, 58.8)
- moved D32 332.3 mm to (-75.0, 21.7)
- moved D28 327.6 mm to (-68.4, 76.0)
- moved D14 316.9 mm to (-62.1, 44.0)
- moved D7 313.2 mm to (-65.1, 64.5)
- moved D27 292.8 mm to (-65.1, 81.8)
- moved D20 285.0 mm to (-65.1, 76.0)
- moved D13 277.2 mm to (-58.4, 76.0)
- moved D31 276.7 mm to (-71.8, 76.0)
- moved D6 274.8 mm to (-65.1, 58.8)
- moved D19 253.1 mm to (-71.8, 70.3)
- moved D26 252.3 mm to (-61.7, 87.5)
- moved D12 248.4 mm to (-72.4, 47.0)
- moved D5 236.2 mm to (-61.7, 64.5)
- moved D18 214.5 mm to (-71.8, 64.5)
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Connections:
- D1 pad 1: Net-(D1-Pad1) -> row0
- D10 pad 1: Net-(D10-Pad1) -> row0
- D11 pad 1: Net-(D11-Pad1) -> row0
- D12 pad 1: Net-(D12-Pad1) -> row0
- D13 pad 1: Net-(D13-Pad1) -> row0
- D14 pad 1: Net-(D14-Pad1) -> row1
- D15 pad 1: Net-(D15-Pad1) -> row1
- D16 pad 1: Net-(D16-Pad1) -> row1
- D17 pad 1: Net-(D17-Pad1) -> row1
- D18 pad 1: Net-(D18-Pad1) -> row1
- D19 pad 1: Net-(D19-Pad1) -> row1
- D2 pad 1: Net-(D2-Pad1) -> row0
- D20 pad 1: Net-(D20-Pad1) -> row1
- D21 pad 1: Net-(D21-Pad1) -> row1
- D22 pad 1: Net-(D22-Pad1) -> row1
- D23 pad 1: Net-(D23-Pad1) -> row1
- D24 pad 1: Net-(D24-Pad1) -> row1
- D25 pad 1: Net-(D25-Pad1) -> row1
- D26 pad 1: Net-(D26-Pad1) -> row1
- D27 pad 1: Net-(D27-Pad1) -> row1
- D28 pad 1: Net-(D28-Pad1) -> row1
- D29 pad 1: Net-(D29-Pad1) -> row2
- D3 pad 1: Net-(D3-Pad1) -> row0
- D30 pad 1: Net-(D30-Pad1) -> row2
- D31 pad 1: Net-(D31-Pad1) -> row2
- D32 pad 1: Net-(D32-Pad1) -> row2
- D4 pad 1: Net-(D4-Pad1) -> row0
- D5 pad 1: Net-(D5-Pad1) -> row0
- D6 pad 1: Net-(D6-Pad1) -> row0
- D7 pad 1: Net-(D7-Pad1) -> row0
- D8 pad 1: Net-(D8-Pad1) -> row0
- D9 pad 1: Net-(D9-Pad1) -> row0
- K_1 pad 1: col1 -> Net-(D1-Pad2)
- K_1 pad 2: Net-(D1-Pad1) -> col0
- K_10 pad 1: col10 -> Net-(D10-Pad2)
- K_10 pad 2: Net-(D6-Pad2) -> col9
- K_11 pad 1: col11 -> Net-(D11-Pad2)
- K_11 pad 2: Net-(D6-Pad1) -> col10
- K_12 pad 1: col12 -> Net-(D12-Pad2)
- K_12 pad 2: Net-(D7-Pad2) -> col11
- K_13 pad 1: col13 -> Net-(D13-Pad2)
- K_13 pad 2: Net-(D7-Pad1) -> col12
- K_2 pad 1: col2 -> Net-(D2-Pad2)
- K_2 pad 2: Net-(D2-Pad2) -> col1
- K_3 pad 1: col3 -> Net-(D3-Pad2)
- K_3 pad 2: Net-(D2-Pad1) -> col2
- K_4 pad 1: col4 -> Net-(D4-Pad2)
- K_4 pad 2: Net-(D3-Pad2) -> col3
- K_5 pad 1: col5 -> Net-(D5-Pad2)
- K_5 pad 2: Net-(D3-Pad1) -> col4
- K_6 pad 1: col6 -> Net-(D6-Pad2)
- K_6 pad 2: Net-(D4-Pad2) -> col5
- K_7 pad 1: col7 -> Net-(D7-Pad2)
- K_7 pad 2: Net-(D4-Pad1) -> col6
- K_8 pad 1: col8 -> Net-(D8-Pad2)
- K_8 pad 2: Net-(D5-Pad2) -> col7
- K_9 pad 1: col9 -> Net-(D9-Pad2)
- K_9 pad 2: Net-(D5-Pad1) -> col8
- U1 pad 18: Net-(U1-Pad18) -> I2C_SCL
- U1 pad 19: Net-(U1-Pad19) -> I2C_SDA
Routing:
- removed copper zone on B.Cu, net GND
- removed copper zone on F.Cu, net GND
Other:
- board size 285 x 94.6 mm -> 304.8 x 119.1 mm

Commit message: Layout Diodes
Parts:
- moved D77 125.3 mm to (-1.59, 113.5)
- moved D47 103.4 mm to (-1.59, 88.1)
- moved D46 99.1 mm to (-4.76, 88.1)
- moved D54 98.8 mm to (-11.1, 96.8)
- moved D40 96.1 mm to (7.94, 80.2)
- moved D45 95.1 mm to (-7.94, 88.1)
- moved D73 94.1 mm to (-14.3, 113.5)
- moved D39 91.0 mm to (4.76, 80.2)
- moved D59 86.4 mm to (4.76, 96.8)
- moved D41 83.8 mm to (-20.6, 88.1)
- moved D32 82.1 mm to (-17.5, 80.2)
- moved D80 79.8 mm to (7.94, 113.5)
- moved D60 79.8 mm to (7.94, 96.8)
- moved D69 78.5 mm to (4.76, 104.8)
- moved D30 77.1 mm to (7.94, 71.4)
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Routing:
- added copper zone on B.Cu, net GND
- added copper zone on F.Cu, net GND
Other:
- board size 304.8 x 119.1 mm -> 341.3 x 119.1 mm

Commit message: Layout Diodes + Route Cols
Parts:
- moved D82 302.4 mm to (297.7, 121.4)
- moved D81 286.5 mm to (278.6, 121.4)
- moved C1 43.2 mm to (-7.30, 34.8)
- moved U1 43.2 mm to (-5.56, 44.5)
- moved R2 43.0 mm to (-2.05, 53.8)
- moved C5 42.6 mm to (-5.55, 34.8)
- moved C3 42.4 mm to (-15.8, 41.1)
- moved C4 42.4 mm to (4.42, 41.1)
- moved Y1 42.4 mm to (-15.9, 44.0)
- moved C2 39.7 mm to (-9.16, 53.8)
- moved R1 34.2 mm to (-15.8, 34.1), turned to 0 degrees
- moved D1 29.9 mm to (7.94, 63.5)
- moved D10 29.9 mm to (-20.6, 63.5)
- moved D11 29.9 mm to (7.94, 71.4)
- moved D20 29.9 mm to (-20.6, 71.4)
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Routing:
- net col8: track 0.00 -> 131.2 mm
- net col11: track 0.00 -> 129.8 mm
- net col6: track 0.00 -> 128.8 mm
- net col10: track 0.00 -> 128.4 mm
- net col12: track 0.00 -> 127.3 mm
- net col1: track 0.00 -> 126.8 mm
- net col9: track 0.00 -> 126.3 mm
- net col2: track 0.00 -> 122.1 mm
- net col0: track 0.00 -> 116.6 mm
- net col7: track 0.00 -> 93.9 mm
- net col5: track 0.00 -> 93.9 mm
- net col4: track 0.00 -> 92.0 mm
- net col3: track 0.00 -> 92.0 mm
- net col14: track 0.00 -> 76.2 mm
- net col13: track 0.00 -> 39.9 mm

Commit message: Diodes
Parts:
- C1, C2, C3, C4, C5, ESD1, F1, R1, R2, R3, R4, R5, R6, SW1, USB1, Y1: moved to B.Cu
- D1, D10, D11, D12, D13, D14, D15, D16, D17, D18, D19, D2, D20, D21, D22, D23, D24, D25, D26, D27, D28, D29, D3, D30, D31, D32, D33, D34, D35, D36, D37, D38, D39, D4, D40, D41, D42, D43, D44, D45, D46, D47, D48, D49, D5, D50, D51, D52, D53, D54, D55, D56, D57, D58, D59, D6, D60, D61, D62, D63, D64, D65, D66, D67, D68, D69, D7, D70, D71, D72, D73, D74, D75, D76, D77, D78, D79, D8, D80, D81, D82, D9: footprint Custom_Footprints:D_SOD-123_Annotated -> Diode_SMD:D_0603_1608Metric_Pad1.05x0.95mm_HandSolder; moved to B.Cu
- U1: value ATmega32U4-AU -> ATmega32U4-MU; footprint Custom_Footprints:ATMEGA32U4_Annotated -> Package_DFN_QFN:QFN-44-1EP_7x7mm_P0.5mm_EP5.2x5.2mm; moved to B.Cu
- moved D28 320.1 mm to (304.0, 46.0)
- moved D58 319.0 mm to (304.0, 84.1)
- moved D57 308.7 mm to (296.9, 84.1)
- moved D43 304.1 mm to (304.0, 65.1)
- moved D72 299.8 mm to (304.0, 103.2)
- moved D80 286.5 mm to (265.9, 122.2)
- moved D56 281.8 mm to (273.1, 84.1)
- moved D70 279.6 mm to (258.8, 103.2)
- moved D27 279.1 mm to (265.9, 46.0)
- moved D71 277.7 mm to (285.0, 103.2)
- moved D42 277.3 mm to (280.2, 65.1)
- moved D13 264.2 mm to (261.1, 22.2)
- moved D79 259.6 mm to (242.1, 122.2)
- moved D40 259.1 mm to (237.3, 65.1)
- moved D26 257.1 mm to (246.9, 46.0)
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Routing:
- net row1: track 0.00 -> 285.8 mm
- net row5: track 0.00 -> 283.4 mm
- net row3: track 0.00 -> 283.4 mm
- net row2: track 0.00 -> 281.0 mm
- net row4: track 0.00 -> 273.8 mm
- net row0: track 0.00 -> 242.9 mm
- net Net-(D57-Pad2): track 0.00 -> 53.8 mm, vias 0 -> 2
- net Net-(D27-Pad2): track 0.00 -> 13.8 mm
- net Net-(D44-Pad2): track 0.00 -> 9.07 mm
- net Net-(D79-Pad2): track 0.00 -> 9.07 mm
- net Net-(D77-Pad2): track 0.00 -> 9.07 mm
- net col2: track 122.1 -> 115.7 mm
- net col12: track 127.3 -> 121.1 mm
- net col0: track 116.6 -> 111.6 mm
- net Net-(D43-Pad2): track 0.00 -> 4.31 mm
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Other:
- board size 341.3 x 119.1 mm -> 304.8 x 119.1 mm

Commit message: Finish
Parts:
- moved C4 126.6 mm to (33.8, 72.9)
- moved C5 123.7 mm to (40.1, 69.2)
- moved R2 123.0 mm to (37.3, 82.0)
- moved U1 122.8 mm to (40.2, 75.7), turned to 270 degrees
- moved C2 121.1 mm to (42.5, 82.0)
- moved Y1 119.9 mm to (47.2, 75.3)
- moved C3 119.9 mm to (47.1, 72.6)
- moved C1 118.3 mm to (36.1, 69.8), turned to 180 degrees
- moved R1 114.8 mm to (43.8, 56.2)
- moved SW1 114.8 mm to (43.8, 53.8)
- moved ESD1 113.3 mm to (33.6, 17.5)
- moved R5 113.3 mm to (28.9, 14.5)
- moved R6 113.3 mm to (37.9, 14.5)
- moved USB1 113.3 mm to (33.4, 4.56)
- moved R4 113.0 mm to (32.6, 28.0)
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Connections:
- U1 pad 1: Net-(U1-Pad1) -> row2
- U1 pad 10: Net-(U1-Pad10) -> row1
- U1 pad 11: Net-(U1-Pad11) -> col4
- U1 pad 20: Net-(U1-Pad20) -> col3
- U1 pad 21: Net-(U1-Pad21) -> col2
- U1 pad 22: Net-(U1-Pad22) -> col1
- U1 pad 25: Net-(U1-Pad25) -> col14
- U1 pad 26: Net-(U1-Pad26) -> col13
- U1 pad 27: Net-(U1-Pad27) -> col12
- U1 pad 28: Net-(U1-Pad28) -> col11
- U1 pad 29: Net-(U1-Pad29) -> col10
- U1 pad 30: Net-(U1-Pad30) -> col9
- U1 pad 31: Net-(U1-Pad31) -> col8
- U1 pad 32: Net-(U1-Pad32) -> col7
- U1 pad 36: Net-(U1-Pad36) -> col6
- U1 pad 37: Net-(U1-Pad37) -> col5
- U1 pad 38: Net-(U1-Pad38) -> row5
- U1 pad 39: Net-(U1-Pad39) -> row4
- U1 pad 40: Net-(U1-Pad40) -> row3
- U1 pad 41: Net-(U1-Pad41) -> col0
- U1 pad 9: Net-(U1-Pad9) -> row0
Routing:
- net +5V: track 0.00 -> 396.4 mm, vias 0 -> 11
- net I2C_SDA: track 0.00 -> 329.0 mm, vias 0 -> 1
- net I2C_SCL: track 0.00 -> 324.3 mm, vias 0 -> 1
- net col14: track 76.2 -> 358.7 mm
- net col13: track 39.9 -> 320.5 mm, vias 0 -> 1
- net col12: track 121.1 -> 369.2 mm, vias 0 -> 1
- net col11: track 130.2 -> 344.8 mm, vias 0 -> 1
- net col10: track 128.4 -> 326.8 mm, vias 0 -> 1
- net col9: track 124.9 -> 305.4 mm, vias 0 -> 1
- net col8: track 131.2 -> 294.1 mm, vias 0 -> 1
- net col7: track 93.9 -> 238.7 mm, vias 0 -> 1
- net col6: track 128.8 -> 259.4 mm, vias 0 -> 1
- net col5: track 93.9 -> 207.5 mm, vias 0 -> 1
- net col4: track 92.0 -> 167.5 mm, vias 0 -> 3
- net col3: track 92.0 -> 148.1 mm, vias 0 -> 1
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Other:
- board size 304.8 x 119.1 mm -> 304.8 x 123 mm

Commit message: Make Gerbers + add Art
Parts:
- added G***: LOGO, art:Koala_120, B.Cu at (256.2, 84.5)
- added REF**: 20x20MakerMark, Logo:20x20MakerMark, B.Cu at (305.6, 20.1)
Other:
- board text added: "koalafications"
